File: soleil_powerpack.kicad_pcb (KiCad board)
At the start: 4 copper layers, 0 parts

Commit message: finish schematic and layout
Parts:
- added C1: 6p, Capacitor_SMD:C_0603_1608Metric, F.Cu at (151.8, 60.0)
- added C10: 100n, Capacitor_SMD:C_0603_1608Metric, F.Cu at (141.4, 63.0)
- added C11: 100n, Capacitor_SMD:C_0603_1608Metric, F.Cu at (121.8, 65.0)
- added C12: 22u, Capacitor_SMD:C_0805_2012Metric, F.Cu at (147.2, 70.8)
- added C13: 22u, Capacitor_SMD:C_0805_2012Metric, F.Cu at (149.8, 70.8)
- added C14: 22u, Capacitor_SMD:C_0805_2012Metric, F.Cu at (137.6, 70.8)
- added C15: 22u, Capacitor_SMD:C_0805_2012Metric, F.Cu at (140.2, 70.8)
- added C16: 1u, Capacitor_SMD:C_0603_1608Metric, F.Cu at (132.8, 65.8)
- added C17: 1u, Capacitor_SMD:C_0603_1608Metric, F.Cu at (136.1, 65.8)
- added C18: 1u, Capacitor_SMD:C_0603_1608Metric, F.Cu at (130.2, 64.7)
- added C2: 100n, Capacitor_SMD:C_0603_1608Metric, F.Cu at (155.4, 65.3)
- added C3: 100n, Capacitor_SMD:C_0603_1608Metric, F.Cu at (155.4, 60.6)
- added C4: 6p, Capacitor_SMD:C_0603_1608Metric, F.Cu at (151.8, 66.0)
- added C5: 100n, Capacitor_SMD:C_0603_1608Metric, F.Cu at (125.2, 61.3)
- added C6: 100n, Capacitor_SMD:C_0603_1608Metric, F.Cu at (127.7, 60.2)
- added C7: 100n, Capacitor_SMD:C_0603_1608Metric, F.Cu at (166.3, 63.0)
- added C8: 100n, Capacitor_SMD:C_0603_1608Metric, F.Cu at (161.7, 63.0)
- added C9: 100n, Capacitor_SMD:C_0603_1608Metric, F.Cu at (164.0, 60.5)
- added D1: ESD5Z5.0, Diode_SMD:D_SOD-523, F.Cu at (166.5, 71.0)
- added D2: RED, LED_SMD:LED_0603_1608Metric, F.Cu at (119.7, 59.2)
- added D3: ESD5Z5.0, Diode_SMD:D_SOD-523, F.Cu at (158.8, 69.2)
- added D4: ESD5Z5.0, Diode_SMD:D_SOD-523, F.Cu at (129.5, 69.0)
- added H1: M2.5, MountingHole:MountingHole_2.7mm_M2.5_ISO14580, F.Cu at (121.0, 76.5)
- added H2: M2.5, MountingHole:MountingHole_2.7mm_M2.5_ISO14580, F.Cu at (121.0, 53.5)
- added H3: M2.5, MountingHole:MountingHole_2.7mm_M2.5_ISO14580, F.Cu at (179.0, 53.5)
- added H4: M2.5, MountingHole:MountingHole_2.7mm_M2.5_ISO14580, F.Cu at (179.0, 76.5)
- added J1: USB_C_Receptacle_PowerOnly_6P, Connector_USB:USB_C_Receptacle_GCT_USB4125-xx-x_6P_TopMnt_Horizontal, F.Cu at (170.1, 76.5)
- added J2: Raspberry_Pi_2_3, gworkman_connector:RaspberryPi_low_profile_HAT_connector, F.Cu at (150.0, 53.5)
- added J3: ~, gworkman_connector:JST_PH_01x02_SMT_Horizontal, F.Cu at (158.8, 75.3)
- added J4: ~, gworkman_connector:JST_PH_01x02_SMT_Horizontal, F.Cu at (129.5, 75.3)
- added JP1: SolderJumper_2_Open, Jumper:SolderJumper-2_P1.3mm_Open_RoundedPad1.0x1.5mm, F.Cu at (179.0, 62.2)
- added JP2: SolderJumper_2_Open, Jumper:SolderJumper-2_P1.3mm_Open_RoundedPad1.0x1.5mm, F.Cu at (179.0, 64.7)
- added JP3: SolderJumper_2_Open, Jumper:SolderJumper-2_P1.3mm_Open_RoundedPad1.0x1.5mm, F.Cu at (179.0, 67.2)
- added L1: 1u5, gworkman_device:L_Vishay_IHLP-2525, F.Cu at (143.8, 76.2)
- added R1: 5k1, Resistor_SMD:R_0603_1608Metric, F.Cu at (146.2, 63.0)
- added R10: 140k, Resistor_SMD:R_0603_1608Metric, F.Cu at (145.6, 68.0)
- added R11: 10k, Resistor_SMD:R_0603_1608Metric, F.Cu at (136.4, 63.0)
- added R12: 13k, Resistor_SMD:R_0603_1608Metric, F.Cu at (136.1, 60.2)
- added R13: 1k, Resistor_SMD:R_0603_1608Metric, F.Cu at (132.8, 60.2)
- added R2: 5k1, Resistor_SMD:R_0603_1608Metric, F.Cu at (143.8, 60.2)
- added R3: 5k1, Resistor_SMD:R_0603_1608Metric, F.Cu at (169.9, 71.0)
- added R4: 5k1, Resistor_SMD:R_0603_1608Metric, F.Cu at (173.5, 71.0)
- added R5: 5k1, Resistor_SMD:R_0603_1608Metric, F.Cu at (125.2, 64.7)
- added R6: 5k1, Resistor_SMD:R_0603_1608Metric, F.Cu at (127.7, 65.8)
- added R7: 5k1, Resistor_SMD:R_0603_1608Metric, F.Cu at (121.8, 59.2)
- added R8: 5k1, Resistor_SMD:R_0603_1608Metric, F.Cu at (130.2, 61.3)
- added R9: 750k, Resistor_SMD:R_0603_1608Metric, F.Cu at (141.9, 68.0)
- added SW1: SW_Push, Button_Switch_SMD:SW_Push_1P1T_NO_CK_KMR2, F.Cu at (120.7, 70.5)
- added U1: MCP7940N-xMNY, Package_DFN_QFN:DFN-8-1EP_3x2mm_P0.5mm_EP1.36x1.46mm, F.Cu at (155.5, 63.0)
- added U2: XC6192B, gworkman_power:USP-8B06, F.Cu at (127.7, 63.0)
- added U3: LM66200, gworkman_power:Texas_DRL0008A_SOT-583, F.Cu at (164.0, 63.0)
- added U4: ATECC608A-MAHDA, Package_DFN_QFN:DFN-8-1EP_3x2mm_P0.5mm_EP1.3x1.5mm, F.Cu at (143.8, 63.4)
- added U5: DRV5032FC, Package_TO_SOT_THT:TO-92Flat, F.Cu at (119.7, 63.2)
- added U6: MP3423, gworkman_power:MPS_PowerQFN-14_2x2mm, F.Cu at (143.8, 70.8)
- added U7: BQ25185, gworkman_power:Texas_DLH0010A_WSON-10, F.Cu at (133.6, 63.0)
- added Y1: 32.768kHz, Crystal:Crystal_SMD_3215-2Pin_3.2x1.5mm, F.Cu at (151.6, 63.0)
Routing:
- net Net-(JP3-B): track 0.00 -> 74.2 mm, vias 0 -> 2
- net Net-(JP2-A): track 0.00 -> 72.1 mm, vias 0 -> 1
- net /~{POWER_ON}: track 0.00 -> 66.2 mm, vias 0 -> 4
- net +6V: track 0.00 -> 56.0 mm, vias 0 -> 9
- net +5V: track 0.00 -> 54.2 mm, vias 0 -> 6
- net /POWER_OFF: track 0.00 -> 49.4 mm, vias 0 -> 2
- net +3V3: track 0.00 -> 48.7 mm, vias 0 -> 3
- net +4V: track 0.00 -> 44.4 mm, vias 0 -> 7
- net +BATT: track 0.00 -> 38.7 mm, vias 0 -> 2
- net /I2C2_SDA: track 0.00 -> 38.3 mm, vias 0 -> 4
- net /I2C2_SCL: track 0.00 -> 35.1 mm, vias 0 -> 2
- net /5V_EN: track 0.00 -> 27.6 mm, vias 0 -> 2
- net /~{RTC_ALARM}: track 0.00 -> 26.2 mm, vias 0 -> 2
- net VBUS: track 0.00 -> 21.4 mm
- net Net-(D2-A): track 0.00 -> 18.4 mm, vias 0 -> 2
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- added copper zone on F.Cu, net +3V3
- added copper zone on F.Cu, net +4V
- added copper zone on F.Cu, net +5V
- added copper zone on B.Cu, net GND
- added copper zone on F.Cu, net GND
- added copper zone on In1.Cu, net GND
- added copper zone on In2.Cu, net GND
- added copper zone on B.Cu, net Net-(L1-Pad2)
- added copper zone on F.Cu, net Net-(L1-Pad2)
Other:
- board outline added: 65 x 30 mm
- board text added: "6V SOLAR"
- board text added: "BATTERY"
- board text added: "Hall Sensor"
- board text added: "Pushbutton"
- board text added: "RTC Alarm"
- board text added: "Wakeup Sources"
