File: soleil_powerpack.kicad_pcb (KiCad board)
At the start: 4 copper layers, 65 x 30 mm, 56 parts, among them J1 USB_C_Receptacle_PowerOnly_6P, J2 Raspberry_Pi_2_3, SW1 SW_Push, U1 MCP7940N-xMNY, U2 XC6192B, U3 LM66200, U4 ATECC608A-MAHDA, U5 DRV5032FC, U6 MP3423, U7 BQ25185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

Commit message: update layout
Routing:
- net GND: vias 66 -> 92
Changed lines of the file:
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@@
 			(psa4output no)
 			(plotreference yes)
-			(plotvalue yes)
+			(plotvalue no)
 			(plotfptext yes)
 			(plotinvisibletext no)
@@
 			(outputformat 1)
 			(mirror no)
-			(drillshape 1)
+			(drillshape 0)
 			(scaleselection 1)
-			(outputdirectory "")
+			(outputdirectory "outputs/gerbers/")
 		)
 	)
@@
 	(net 59 "Net-(JP3-B)")
 	(footprint "MountingHole:MountingHole_2.7mm_M2.5_ISO14580"
-		(locked yes)
 		(layer "F.Cu")
 		(at 121 53.5)
@@
 	)
 	(footprint "gworkman_connector:RaspberryPi_low_profile_HAT_connector"
-		(locked yes)
 		(layer "F.Cu")
 		(at 150 53.5)
@@
 	)
 	(footprint "MountingHole:MountingHole_2.7mm_M2.5_ISO14580"
-		(locked yes)
 		(layer "F.Cu")
 		(at 179 76.5)
@@
 	)
 	(footprint "MountingHole:MountingHole_2.7mm_M2.5_ISO14580"
-		(locked yes)
 		(layer "F.Cu")
 		(at 179 53.5)
@@
 	)
 	(footprint "MountingHole:MountingHole_2.7mm_M2.5_ISO14580"
-		(locked yes)
 		(layer "F.Cu")
 		(at 121 76.5)
@@
 	)
 	(via
+		(at 142.8 73.5)
+		(size 0.6)
+		(drill 0.3)
+		(layers "F.Cu" "B.Cu")
+		(free yes)
+		(net 2)
+	)
+	(via
+		(at 144.8 78.5)
+		(size 0.6)
+		(drill 0.3)
+		(layers "F.Cu" "B.Cu")
+		(free yes)
+		(net 2)
+	)
+	(via
 		(at 166.5 60.5)
 		(size 0.6)
@@
 	)
 	(via
+		(at 121.8 61.5)
+		(size 0.6)
+		(drill 0.3)
+		(layers "F.Cu" "B.Cu")
+		(free yes)
+		(net 2)
+	)
+	(via
+		(at 151.7 78.5)
+		(size 0.6)
+		(drill 0.3)
+		(layers "F.Cu" "B.Cu")
+		(free yes)
+		(net 2)
+	)
+	(via
 		(at 134.5 53.5)
 		(size 0.6)
@@
 	)
 	(via
+		(at 156 69.8)
+		(size 0.6)
+		(drill 0.3)
+		(layers "F.Cu" "B.Cu")
+		(free yes)
+		(net 2)
+	)
+	(via
 		(at 136.1 70)
 		(size 0.6)
@@
 	)
 	(via
+		(at 164 66)
+		(size 0.6)
+		(drill 0.3)
+		(layers "F.Cu" "B.Cu")
+		(free yes)
+		(net 2)
+	)
+	(via
+		(at 142.8 78.5)
+		(size 0.6)
+		(drill 0.3)
+		(layers "F.Cu" "B.Cu")
+		(free yes)
+		(net 2)
+	)
+	(via
 		(at 172.5 77.5)
 		(size 0.6)
@@
 	)
 	(via
+		(at 159.8 76)
+		(size 0.6)
+		(drill 0.3)
+		(layers "F.Cu" "B.Cu")
+		(free yes)
+		(net 2)
+	)
+	(via
 		(at 129.175003 66.8)
 		(size 0.45)
@@
 	)
 	(via
+		(at 151.7 76)
+		(size 0.6)
+		(drill 0.3)
+		(layers "F.Cu" "B.Cu")
+		(free yes)
+		(net 2)
+	)
+	(via
 		(at 126.5 70)
 		(size 0.6)
@@
 	)
 	(via
+		(at 148.7 78.5)
+		(size 0.6)
+		(drill 0.3)
+		(layers "F.Cu" "B.Cu")
+		(free yes)
+		(net 2)
+	)
+	(via
 		(at 133.5 70)
 		(size 0.6)
@@
 	)
 	(via
+		(at 157.7 76)
+		(size 0.6)
+		(drill 0.3)
+		(layers "F.Cu" "B.Cu")
+		(free yes)
+		(net 2)
+	)
+	(via
 		(at 158.15 64.400002)
 		(size 0.45)
@@
 	)
 	(via
-		(at 170 77.5)
+		(at 170.1 77.5)
 		(size 0.6)
 		(drill 0.3)
@@
 	)
 	(via
+		(at 152.5 71.7)
+		(size 0.6)
+		(drill 0.3)
+		(layers "F.Cu" "B.Cu")
+		(free yes)
+		(net 2)
+	)
+	(via
 		(at 145.7 59.500003)
 		(size 0.45)
@@
 	)
 	(via
+		(at 162.7 61.6)
+		(size 0.6)
+		(drill 0.3)
+		(layers "F.Cu" "B.Cu")
+		(free yes)
+		(net 2)
+	)
+	(via
 		(at 145.7 60.9)
 		(size 0.45)
@@
 	)
 	(via
+		(at 155.5 61.5)
+		(size 0.6)
+		(drill 0.3)
+		(layers "F.Cu" "B.Cu")
+		(free yes)
+		(net 2)
+	)
+	(via
+		(at 158.2 60.6)
+		(size 0.6)
+		(drill 0.3)
+		(layers "F.Cu" "B.Cu")
+		(free yes)
+		(net 2)
+	)
+	(via
 		(at 152.5 67.5)
 		(size 0.6)
@@
 	)
 	(via
-		(at 158.6 62.549997)
-		(size 0.45)
-		(drill 0.25)
+		(at 142.8 76)
+		(size 0.6)
+		(drill 0.3)
 		(layers "F.Cu" "B.Cu")
 		(free yes)
@@
 	)
 	(via
-		(at 167.5 77.5)
+		(at 167.7 77.5)
+		(size 0.6)
+		(drill 0.3)
+		(layers "F.Cu" "B.Cu")
+		(free yes)
+		(net 2)
+	)
+	(via
+		(at 149.8 61.7)
+		(size 0.6)
+		(drill 0.3)
+		(layers "F.Cu" "B.Cu")
+		(free yes)
+		(net 2)
+	)
+	(via
+		(at 157.7 78.5)
 		(size 0.6)
 		(drill 0.3)
@@
 	)
 	(via
+		(at 148.7 76)
+		(size 0.6)
+		(drill 0.3)
+		(layers "F.Cu" "B.Cu")
+		(free yes)
+		(net 2)
+	)
+	(via
 		(at 137.5 78.5)
 		(size 0.6)
@@
 	)
 	(via
+		(at 167.3 75.5)
+		(size 0.6)
+		(drill 0.3)
+		(layers "F.Cu" "B.Cu")
+		(free yes)
+		(net 2)
+	)
+	(via
 		(at 144.5 53.5)
 		(size 0.6)
@@
 	)
 	(via
+		(at 159.8 78.5)
+		(size 0.6)
+		(drill 0.3)
+		(layers "F.Cu" "B.Cu")
+		(free yes)
+		(net 2)
+	)
+	(via
 		(at 137 53.5)
 		(size 0.6)
@@
 	)
 	(via
+		(at 124.4 78.5)
+		(size 0.6)
+		(drill 0.3)
+		(layers "F.Cu" "B.Cu")
+		(free yes)
+		(net 2)
+	)
+	(via
+		(at 152.5 69.8)
+		(size 0.6)
+		(drill 0.3)
+		(layers "F.Cu" "B.Cu")
+		(free yes)
+		(net 2)
+	)
+	(via
 		(at 165 53.5)
 		(size 0.6)
@@
 	)
 	(via
+		(at 136.1 61.2)
+		(size 0.6)
+		(drill 0.3)
+		(layers "F.Cu" "B.Cu")
+		(free yes)
+		(net 2)
+	)
+	(via
 		(at 149 67.5)
 		(size 0.6)
@@
 	)
 	(via
+		(at 144.8 76)
+		(size 0.6)
+		(drill 0.3)
+		(layers "F.Cu" "B.Cu")
+		(free yes)
+		(net 2)
+	)
+	(via
 		(at 139.5 63)
 		(size 0.6)
@@
 	)
 	(via
+		(at 147.1 68.7)
+		(size 0.6)
+		(drill 0.3)
+		(layers "F.Cu" "B.Cu")
+		(free yes)
+		(net 2)
+	)
+	(via
 		(at 170 53.5)
 		(size 0.6)
 		(drill 0.3)
+		(layers "F.Cu" "B.Cu")
+		(free yes)
+		(net 2)
+	)
+	(via
+		(at 172.9 75.5)
+		(size 0.6)
+		(drill 0.3)
