File: soleil_powerpack.kicad_sch (KiCad schematic)
At the start: 48 parts, among them J1 Raspberry_Pi_2_3, J2 USB_C_Receptacle_PowerOnly_6P, SW1 SW_Push, U1 MCP7940N-xMNY, U2 BQ25185, U3 MS3423, U4 LM66200, U5 XC6192, U6 DRV5032FC, U7 ATECC608A-MAHDA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

Commit message: finish schematic and layout
Parts:
- removed JP1, JP2, JP3: SolderJumper_2_Bridged, symbol Jumper:SolderJumper_2_Bridged
- added C6: 100n, Capacitor_SMD:C_0603_1608Metric, symbol Device:C_Small
- added H1, H2, H3, H4: M2.5, MountingHole:MountingHole_2.7mm_M2.5_ISO14580, symbol Mechanical:MountingHole
- added JP1, JP2, JP3: SolderJumper_2_Open, Jumper:SolderJumper-2_P1.3mm_Open_RoundedPad1.0x1.5mm, symbol Jumper:SolderJumper_2_Open
- added R1, R2: 5k1, Resistor_SMD:R_0603_1608Metric, symbol Device:R_Small
- added R11: 10k, Resistor_SMD:R_0603_1608Metric, symbol Device:R_Small
- C1, C3, C8: footprint (none) -> Capacitor_SMD:C_0603_1608Metric
- C10: renamed from C17; footprint (none) -> Capacitor_SMD:C_0603_1608Metric
- C11: renamed from C16; footprint (none) -> Capacitor_SMD:C_0603_1608Metric
- C16: renamed from C7; footprint (none) -> Capacitor_SMD:C_0603_1608Metric
- C17: renamed from C5; footprint (none) -> Capacitor_SMD:C_0603_1608Metric
- C18: renamed from C6; footprint (none) -> Capacitor_SMD:C_0603_1608Metric
- C2: renamed from C4; footprint (none) -> Capacitor_SMD:C_0603_1608Metric
- C4: renamed from C2; footprint (none) -> Capacitor_SMD:C_0603_1608Metric
- C5: renamed from C15; footprint (none) -> Capacitor_SMD:C_0603_1608Metric
- C7: renamed from C9; footprint (none) -> Capacitor_SMD:C_0603_1608Metric
- C9: renamed from C10; footprint (none) -> Capacitor_SMD:C_0603_1608Metric
- D1: renamed from D2; LCSC (none) -> C2905624
- D2: renamed from D1; footprint (none) -> LED_SMD:LED_0603_1608Metric
- D3, D4: LCSC (none) -> C2905624
- J1: renamed from J2; footprint (none) -> Connector_USB:USB_C_Receptacle_GCT_USB4125-xx-x_6P_TopMnt_Horizontal; DigiKey (none) -> 2073-USB4125-GF-ACT-ND; MPN (none) -> USB4125-GF-A
- J2: renamed from J1; footprint (none) -> gworkman_connector:RaspberryPi_low_profile_HAT_connector; DigiKey (none) -> 612-HLE-120-02-F-DV-BE-A-ND; LCSC (none) -> C2685112; MPN (none) -> HLE-120-02-F-DV-BE-A
- J3, J4: footprint (none) -> gworkman_connector:JST_PH_01x02_SMT_Horizontal; DigiKey (none) -> 455-S2B-PH-SM4-TBCT-ND; LCSC (none) -> C295747; MPN (none) -> S2B-PH-SM4-TB
- L1: footprint Inductor_SMD:L_Vishay_IHLP-2525 -> gworkman_device:L_Vishay_IHLP-2525; LCSC (none) -> C845020
- R10: renamed from R4; footprint (none) -> Resistor_SMD:R_0603_1608Metric
- R12: renamed from R2; footprint (none) -> Resistor_SMD:R_0603_1608Metric
- R13: renamed from R1; footprint (none) -> Resistor_SMD:R_0603_1608Metric
- R3: renamed from R10; footprint (none) -> Resistor_SMD:R_0603_1608Metric
- R4: renamed from R9; footprint (none) -> Resistor_SMD:R_0603_1608Metric
- R5: footprint (none) -> Resistor_SMD:R_0603_1608Metric
- R6: renamed from R8; footprint (none) -> Resistor_SMD:R_0603_1608Metric
- R7: renamed from R6; footprint (none) -> Resistor_SMD:R_0603_1608Metric
- R8: renamed from R7; footprint (none) -> Resistor_SMD:R_0603_1608Metric
- R9: renamed from R3; footprint (none) -> Resistor_SMD:R_0603_1608Metric
- SW1: footprint (none) -> Button_Switch_SMD:SW_Push_1P1T_NO_CK_KMR2; DigiKey (none) -> 401-1428-1-ND; LCSC (none) -> C221678; MPN (none) -> KMR223GLFG
- U1: LCSC (none) -> C623889
- U2: renamed from U5; value XC6192 -> XC6192B; LCSC (none) -> C2442364
- U3: renamed from U4; LCSC (none) -> C3235556
- U4: renamed from U7; DigiKey (none) -> ATECC608A-MAHDA-SCT-ND; LCSC (none) -> C616908; MPN (none) -> ATECC608A-MAHDA-S
- U5: renamed from U6; LCSC (none) -> C2866256
- U6: renamed from U3; value MS3423 -> MP3423; LCSC (none) -> C2682483
- U7: renamed from U2; LCSC (none) -> C19725033
- Y1: LCSC (none) -> C276424
- renumbered C11 to C13, C13 to C14, C14 to C15
Connections:
- net +3V3: now also J2.1 (3V3), J2.17 (3V3), R1.1, R2.1
- net +5V: now also J2.2 (5V), J2.4 (5V)
- net GND: now also C6.2, R11.2
- net I2C2_SCL: now also R2.2
- net I2C2_SDA: now also R1.2
- net ~{POWER_ON}: now also JP1.1 (A), JP2.2 (B), JP3.1 (A)
- net ~{RTC_ALARM}: now also JP1.2 (B)
- net at SW1.1: now also JP3.2 (B)
- net at D2.2 (A), R6.2, U2.8 (VOUT): now also C6.1
- net at U5.3 (OUT): now also JP2.1 (A)
- net BATT_CHRG_STAT1: no longer names the net of U7.9 (STAT1)
- net BATT_CHRG_STAT2: no longer names the net of U7.3 (STAT2)
- net BATT_NTC: no longer names the net of U7.6 (TS/MR)
- net BATT_NTC: now also R11.1
- no-connect marks 1 -> 28
Other:
- note added: "- 925nA Iq on battery backup - I2C address 0x6F"
- note added: "- Input 1.6V - 5.5V - Up to 2.5A per channel - 1.32uA Iq"
- note added: "- Iq 10nA in shutdown"
- note added: "- Open drain interrupts, pull up on ~{POWER_ON} load switch pin"
- note added: "- Output 5.13V, 3A - 0.807*(1+R1/R2) - R1 > 600k - Low ESR caps"
- note added: "- USB-C charger, JST PH for battery and solar - Battery cable compatible with Adafruit 1S lipo batteries"
- note added: "- compatible with NervesKey for connection to NervesHub"
- note added: "- input current limit of 1A - charge voltage 4.2V - fast charge 500mA - stat pins OD"
- note added: "5V Boost Converter"
- note added: "Battery Charger"
- note added: "Certificate Storage"
- note added: "Connectors"
- note added: "Ideal Diode"
- note added: "Load Switch"
- note added: "Mounting Holes"
- note added: "Raspberry Pi"
- note added: "Real Time Clock"
- note added: "Wakeup Sources"
- moved on the sheet: C1, C10, C11, C12, C13, C14, C15, C16, C17, C18, C2, C3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
