File: power.kicad_sch (KiCad schematic)
At the start: 51 parts, among them J1 USB_C_Receptacle_PowerOnly_6P, U2 XC6192B, U3 LM66200, U6 MP3423, U7 BQ25185, U8 TLV76701DRVx, U9 BQ27427

Commit message: add digikey part numbers
Parts:
- C12, C13, C14, C15: DigiKey (none) -> 1276-6780-1-ND; MPN (none) -> CL21A226MOCLRNC
- C16, C17, C18, C21, C23, C24: DigiKey (none) -> 1276-1067-1-ND; MPN (none) -> CL05A105KO5NNNC
- C19, C20, C22: DigiKey (none) -> 490-10012-1-ND; MPN (none) -> GRM155C80J225KE95D
- C5, C6, C7, C8, C9: DigiKey (none) -> 490-6328-1-ND; LCSC (none) -> C71629; MPN (none) -> GRM155R71C104KA88J
- D2, D5: DigiKey (none) -> 1497-1174-1-ND; MPN (none) -> XZMDK68W-2
- R10: DigiKey (none) -> YAG2978CT-ND; MPN (none) -> RC0402FR-07140KL
- R11, R16, R17, R19, R6: DigiKey (none) -> 1276-3431-1-ND; MPN (none) -> RC1005F103CS
- R12: DigiKey (none) -> 311-13.0KLRCT-ND; MPN (none) -> RC0402FR-0713KL
- R13: DigiKey (none) -> 311-1.0KJRCT-ND; MPN (none) -> RC0402JR-071KL
- R14: DigiKey (none) -> YAG5649CT-ND; MPN (none) -> AC0402FR-071M2L
- R15: DigiKey (none) -> RMCF0402FT200KCT-ND; MPN (none) -> RMCF0402FT200K
- R18, R3, R4, R5, R7, R8: DigiKey (none) -> 2019-RK73B1ETTP512JCT-ND; MPN (none) -> RK73B1ETTP512J
- R9: DigiKey (none) -> YAG3228CT-ND; MPN (none) -> RC0402FR-07750KL
- U2: DigiKey 893-XC6193BANNER-GCT-ND -> 893-1413-1-ND; LCSC C2442364 -> (none); MPN XC6193BANNER-G -> XC6192BANNER-G
- U9: DigiKey (none) -> 296-BQ27427YZFRCT-ND; MPN (none) -> BQ27427YZFR

Commit message: clean and plot schematic to pdf
Parts:
- D3: value ESD5Z6.0 -> ESD5Z24; DigiKey ESD5Z6.0T1GOSCT-ND -> 4878-ESD5Z24CT-ND; LCSC C2890110 -> C23380859; MPN ESD5Z6.0T1G -> ESD5Z24
Other:
- moved on the sheet: C12, C13, C14, C15, C19, C20, C24, C5, C6, C7, C8, C9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

Commit message: add readme
Other:
- note added: "- Input current limit of 1A - Charge voltage 4.2V - Fast charge current 500mA - Battery-only mode 4uA Iq"
- note removed: "- Input current limit of 1A - Charge voltage 4.2V - Fast charge current 500mA"
Changed lines of the file:
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@@
 		)
 	)
-	(text "- Input current limit of 1A\n- Charge voltage 4.2V\n- Fast charge current 500mA\n"
+	(text "- Input current limit of 1A\n- Charge voltage 4.2V\n- Fast charge current 500mA\n- Battery-only mode 4uA Iq\n"
 		(exclude_from_sim no)
 		(at 187.96 21.59 0)

Commit message: update schematic for publish
Parts:
- removed C12, C13, C14, C15: 22u, Capacitor_SMD:C_0805_2012Metric, symbol Device:C_Small
- removed C16, C17, C18, C21, C23, C24: 1u, Capacitor_SMD:C_0402_1005Metric, symbol Device:C_Small
- removed C19, C20, C22: 2u2, Capacitor_SMD:C_0402_1005Metric, symbol Device:C_Small
- removed C5, C6, C7, C8, C9: 100n, Capacitor_SMD:C_0402_1005Metric, symbol Device:C_Small
- removed D1, D4: ESD5Z6.0, Diode_SMD:D_SOD-523, symbol Diode:ESD5Zxx
- removed D2, D5: RED, LED_SMD:LED_0402_1005Metric, symbol Device:LED_Small
- removed D3: ESD5Z24, Diode_SMD:D_SOD-523, symbol Diode:ESD5Zxx
- removed J1: USB_C_Receptacle_PowerOnly_6P, Connector_USB:USB_C_Receptacle_GCT_USB4125-xx-x_6P_TopMnt_Horizontal, symbol Connector:USB_C_Receptacle_PowerOnly_6P
- removed J3, J4: ~, gworkman_connector:JST_PH_01x02_SMT_Horizontal, symbol Connector_Generic:Conn_01x02
- removed JP4: SolderJumper_2_Open, Jumper:SolderJumper-2_P1.3mm_Open_RoundedPad1.0x1.5mm, symbol Jumper:SolderJumper_2_Open
- removed L1: 1u5, gworkman_device:L_Vishay_IHLP-2525, symbol Device:L_Small
- removed R10: 140k, Resistor_SMD:R_0402_1005Metric, symbol Device:R_Small
- removed R11, R16, R17, R19, R6: 10k, Resistor_SMD:R_0402_1005Metric, symbol Device:R_Small
- removed R12: 13k, Resistor_SMD:R_0402_1005Metric, symbol Device:R_Small
- removed R13: 1k, Resistor_SMD:R_0402_1005Metric, symbol Device:R_Small
- removed R14: 1M2, Resistor_SMD:R_0402_1005Metric, symbol Device:R_Small
- removed R15: 200k, Resistor_SMD:R_0402_1005Metric, symbol Device:R_Small
- removed R18, R3, R4, R5, R7, R8: 5k1, Resistor_SMD:R_0402_1005Metric, symbol Device:R_Small
- removed R9: 750k, Resistor_SMD:R_0402_1005Metric, symbol Device:R_Small
- removed U2: XC6192B, gworkman_power:USP-8B06, symbol gworkman_power:XC6192
- removed U3: LM66200, gworkman_power:Texas_DRL0008A_SOT-583, symbol gworkman_power:LM66200
- removed U6: MP3423, gworkman_power:MPS_PowerQFN-14_2x2mm, symbol gworkman_power:MP3423
- removed U7: BQ25185, gworkman_power:Texas_DLH0010A_WSON-10, symbol gworkman_power:BQ25185
- removed U8: TLV76701DRVx, Package_SON:WSON-6-1EP_2x2mm_P0.65mm_EP1x1.6mm_ThermalVias, symbol Regulator_Linear:TLV76701DRVx
- removed U9: BQ27427, Package_BGA:Texas_DSBGA-9_1.62mmx1.58mm_Layout3x3_P0.5mm, symbol gworkman_power:BQ27427
Connections:
- no-connect marks 2 -> 0
Other:
- note removed: "- Input 1.6V - 5.5V - Up to 2.5A per channel - 1.32uA Iq"
- note removed: "- Input current limit of 1A - Charge voltage 4.2V - Fast charge current 500mA - Battery-only mode 4uA Iq"
- note removed: "- Integrated sense resistor - 50uA in normal mode, 9uA in sleep mode - Auto sleep mode when low current (< 10mA) - I2C address 0x55 - Lowpass filter on GPOUT to prevent disabling the system on SOC updates (1-ms pulse low) - RC time constant of 10ms"
- note removed: "- Iq 10nA in shutdown - ~{POWER_ON} pull low to wake from sleep - Pulse SHDN high to enter sleep mode"
- note removed: "- Output 5.13V, 3A - 0.807*(1+R1/R2) - R1 > 600k - Low ESR caps - EN high when > 1.2V"
- note removed: "- USB-C charger, JST PH for battery and solar - Battery cable compatible with Adafruit 1S lipo batteries - DC_IN optimized for 6V, 1.5W solar panel - DC_IN can be used with any DC power source up to 16V"
- note removed: "- VDC set point to 5.6V - VDC tracks DC_IN when DC_IN < 5.6 + V_DO - V_DO is 0.4V @ 500mA - VDC 2.5V - 16V - Iout up to 1A - Iq is 50 uA (1.5uA in shutdown)"
- note removed: "5V Boost Converter"
- note removed: "Battery Charger"
- note removed: "Battery Fuel Gauge"
- note removed: "Connectors"
- note removed: "Linear Regulator"
- note removed: "Load Switch"
- note removed: "Power Multiplexer"
