File: boost_converter.kicad_sch (KiCad schematic)
At the start: 9 parts, among them U6 MP3423

Commit message: finish all schematic changes
Parts:
- added D2: RED, LED_SMD:LED_0402_1005Metric, symbol Device:LED_Small
- added D6: 500mV @ 2A, Diode_SMD:D_SOD-123F, symbol Device:D_Schottky_Small
- added R7: 10k, Resistor_SMD:R_0402_1005Metric, symbol Device:R_Small
- R10: value 140k -> 133k; DigiKey YAG2978CT-ND -> YAG2970CT-ND; LCSC C114151 -> C327374; MPN RC0402FR-07140KL -> RC0402FR-07133KL
Connections:
- net 5V: now also D6.1 (K); no longer C14.1, C15.1, C24.1, R9.1, U6.4 (OUT), U6.5 (OUT), U6.6 (OUT)
- net GND: now also R7.1
- new net: C14.1, C15.1, C24.1, D2.2 (A), D6.2 (A), R9.1, U6.4 (OUT), U6.5 (OUT), U6.6 (OUT)
- new net: D2.1 (K), R7.2
Other:
- moved on the sheet: C12, C13, C14, C15, C24, L1, R10, R9, U6
