File: qwiic.kicad_sch (KiCad schematic)
At the start: 2 parts, among them J5 Conn_01x04

Commit message: finish all schematic changes
Parts:
- J5: value Conn_01x04 -> SM04B-SRSS-TB; DigiKey (none) -> 455-SM04B-SRSS-TBCT-ND; LCSC (none) -> C160404; MPN (none) -> SM04B-SRSS-TB; digikey 455-SM04B-SRSS-TBCT-ND -> (none); lcsc C160404 -> (none); mpn SM04B-SRSS-TB -> (none)
Changed lines of the file:
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@@
 	)
 	(rectangle
-		(start 114.3 55.88)
-		(end 193.04 105.41)
+		(start 110.49 63.5)
+		(end 190.5 107.95)
 		(stroke
 			(width 0)
@@
 	(text "Qwiic Connector"
 		(exclude_from_sim no)
-		(at 114.3 53.34 0)
+		(at 110.49 60.96 0)
 		(effects
 			(font
@@
 		(dnp no)
 		(property "Reference" "J5"
-			(at 172.72 86.3601 0)
+			(at 172.72 83.82 0)
 			(effects
 				(font
@@
 			)
 		)
-		(property "Value" "Conn_01x04"
-			(at 172.72 83.8201 0)
+		(property "Value" "SM04B-SRSS-TB"
+			(at 172.72 86.36 0)
 			(effects
 				(font
@@
 			)
 		)
-		(property "mpn" "SM04B-SRSS-TB"
+		(property "MPN" "SM04B-SRSS-TB"
 			(at 170.18 86.36 0)
 			(effects
@@
 			)
 		)
-		(property "digikey" "455-SM04B-SRSS-TBCT-ND"
+		(property "DigiKey" "455-SM04B-SRSS-TBCT-ND"
 			(at 170.18 86.36 0)
 			(effects
@@
 			)
 		)
-		(property "lcsc" "C160404"
+		(property "LCSC" "C160404"
 			(at 170.18 86.36 0)
 			(effects
@@
 	(symbol
 		(lib_id "Sparkfun-Qwiic:qwiic_Logo")
-		(at 170.18 74.93 0)
+		(at 161.29 71.12 0)
 		(unit 1)
 		(exclude_from_sim no)
@@
 		(fields_autoplaced yes)
 		(property "Reference" "G1"
-			(at 170.18 71.12 0)
+			(at 161.29 67.31 0)
 			(effects
 				(font
@@
 		)
 		(property "Value" "qwiic_Logo"
-			(at 170.18 78.74 0)
+			(at 161.29 74.93 0)
 			(effects
 				(font
@@
 		)
 		(property "Footprint" "Sparkfun-Qwiic:qwiic_5mm"
-			(at 170.18 81.28 0)
+			(at 161.29 77.47 0)
 			(effects
 				(font
@@
 		)
 		(property "Datasheet" ""
-			(at 170.18 74.93 0)
+			(at 161.29 71.12 0)
 			(effects
 				(font
@@
 		)
 		(property "Description" ""
-			(at 170.18 74.93 0)
+			(at 161.29 71.12 0)
 			(effects
 				(font
