File: raspberry_pi.kicad_sch (KiCad schematic)
At the start: 11 parts, among them J2 Raspberry_Pi, U4 ATECC608A-MAHDA

Commit message: finish all schematic changes
Parts:
- J2: Alternative (none) -> HLE-120-02-F-DV-BE-A; DigiKey 612-HLE-120-02-F-DV-BE-A-ND -> (none); MPN HLE-120-02-F-DV-BE-A -> FH-00339
Changed lines of the file:
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@@
 			)
 		)
-		(property "MPN" "HLE-120-02-F-DV-BE-A"
+		(property "MPN" "FH-00339"
 			(at 99.06 85.09 0)
 			(effects
@@
 			)
 		)
-		(property "DigiKey" "612-HLE-120-02-F-DV-BE-A-ND"
+		(property "DigiKey" ""
 			(at 99.06 85.09 0)
 			(effects
+				(font
+					(size 1.27 1.27)
+				)
+				(hide yes)
+			)
+		)
+		(property "Alternative" "HLE-120-02-F-DV-BE-A"
+			(at 99.06 85.09 0)
+			(effects
